File: OPI CM5 Blade Board/OPI CM5 Blade board.kicad_pcb (KiCad board)
At the start: 4 copper layers, 241.6 x 42.5 mm, 81 parts, among them J1 OPi_CM5_CORE JP1 100PIN, J2 OPi_CM5_CORE JP2 100PIN, J3 OPi_CM5_CORE JP13100PIN, J4 Bus_PCI_Express_x4, J5 J_1-2199230-5, SW1 USER_SW, SW2 RESET_SW, SW3 BOOT_SW, SW4 PWR_SW, U1 SHT40-BD1B-R3, U2 SHT40-BD1B-R3, U4 SM8103ADC, U5 SM8103ADC

Commit message: Project complete
Parts:
- added D1: RED, LED_SMD:LED_0603_1608Metric_Pad1.05x0.95mm_HandSolder, F.Cu at (49.3, 32.6)
- added R1: 560R, Resistor_SMD:R_0201_0603Metric_Pad0.64x0.40mm_HandSolder, F.Cu at (52.3, 32.6)
- moved R13 36.7 mm to (42.1, 31.0)
- moved D11 36.7 mm to (39.1, 31.0)
- moved ED5 28.4 mm to (39.5, 62.3), turned to 180 degrees
- moved D10 27.7 mm to (49.3, 39.2)
- moved R10 27.4 mm to (52.3, 39.2)
- moved NC/SIP1X3 27.0 mm to (39.5, 65.5)
- moved D2 26.6 mm to (45.2, 58.5)
- moved CC1 26.5 mm to (46.7, 58.5)
- moved R2 26.5 mm to (48.0, 58.5)
- moved SW4 26.5 mm to (40.4, 58.5)
- moved U1 25.8 mm to (47.3, 67.6), turned to 180 degrees
- moved R7 25.7 mm to (42.1, 34.3)
- moved D8 25.7 mm to (39.1, 34.3)
- moved R11 25.5 mm to (39.5, 68.2), turned to 180 degrees
- moved R12 25.5 mm to (39.5, 69.5), turned to 180 degrees
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Connections:
- net /HDMI_TX0_SDA_M0 renamed /HDMI0_TX_SDA_M0
- J2 pad 100: /HDMI_TX0_SCL_M0 -> /HDMI0_TX_SCL_M0
- J2 pad 51: /HDMI_TX0_CEC_M0 -> /HDMI0_TX_CEC_M0
- J2 pad 53: /HDMI_TX0_SBDN -> /HDMI0_SBDN
- J2 pad 70: /HDMI_TX0_D2P -> /HDMI0_TX2P
- J2 pad 72: /HDMI_TX0_D2N -> /HDMI0_TX2N
- J2 pad 76: /HDMI_TX0_D1P -> /HDMI0_TX1P
- J2 pad 78: /HDMI_TX0_D1N -> /HDMI0_TX1N
- J2 pad 82: /HDMI_TX0_D0P -> /HDMI0_TX0P
- J2 pad 84: /HDMI_TX0_D0N -> /HDMI0_TX0N
- J2 pad 88: /HDMI_TX0_D3P -> /HDMI0_TX3P
- J2 pad 90: /HDMI_TX0_D3N -> /HDMI0_TX3N
- J3 pad 1: /USB20_HOST1_DP -> /USB20_HOST1_DN
- J3 pad 3: /USB20_HOST1_DN -> /USB20_HOST1_DP
- J4 pad A15: unconnected-(J4-PadA15) -> /GMAC_MDC
- J4 pad A16: /GMAC_MDC -> /GMAC_TXCLK
- J4 pad A17: /GMAC_TXCLK -> GND
- J4 pad B12: /UART_TX -> /UART2_TX
- J4 pad B13: /UART_RX -> /UART2_RX
- J4 pad B15: /USB20_HOST1_DM -> /USB20_HOST1_DN
- J4 pad B18: /HDMI0_TX_ON_H -> /HDMI0_TX_CEC_M0
- J4 pad B19: /HDMI_TX0_CEC_M0 -> /HDMI0_SBDN
- J4 pad B20: /HDMI_TX0_SBDN -> /HDMI0_SBDP
- J4 pad B22: /HDMI_TX0_D2P -> /HDMI0_TX_SCL_M0
- J4 pad B23: /HDMI_TX0_D2N -> /HDMI0_TX1P
- J4 pad B24: /HDMI_TX0_D1P -> /HDMI0_TX1N
- J4 pad B25: /HDMI0_TX1N -> /HDMI0_TX3P
- J4 pad B26: /HDMI_TX0_SCL_M0 -> /HDMI0_TX3N
- J4 pad B27: /HDMI_TX0_D3N -> /HDMI0_TX0N
- J4 pad B28: /HDMI_TX0_D3P -> /HDMI0_TX0P
- J4 pad B29: /HDMI_TX0_D0N -> /HDMI0_TX2N
- J4 pad B30: /HDMI_TX0_D0P -> /HDMI0_TX2P
- J4 pad B32: /HDMI0_SBDP -> /HDMI0_TX_ON_H
- R10 pad 1: /TMP_SN2_LED -> +12V
- R11 pad 1: /UART_TX -> /UART2_TX
- R12 pad 1: /UART_RX -> /UART2_RX
- R3 pad 1: VCC_5V0 -> +5V_3A
- U2 pad 3: +3.3V_3A -> /VCC_3V3_S3
Routing:
- net +12V: track 25.6 -> 321.2 mm, vias 0 -> 30
- net +3.3V_3A: track 0.00 -> 271.3 mm
- net /PMIC_RESET_L: track 0.00 -> 270.0 mm, vias 0 -> 3
- net /UART2_RX: track 0.00 -> 258.4 mm, vias 0 -> 2
- net /UART2_TX: track 0.00 -> 258.0 mm, vias 0 -> 2
- net /PWRON_L: track 0.00 -> 256.3 mm, vias 0 -> 2
- net +5V_3A: track 58.9 -> 287.5 mm, vias 0 -> 2
- net /BOOT_KEY: track 0.00 -> 197.3 mm, vias 0 -> 2
- net /USER_KEY: track 0.00 -> 193.8 mm, vias 0 -> 2
- net /USER_LED: track 0.00 -> 185.2 mm, vias 0 -> 2
- net /DEBUG_LED: track 0.00 -> 182.8 mm, vias 0 -> 2
- net /TMP_SN1_LED: track 0.00 -> 180.3 mm, vias 0 -> 2
- net GND: track 13.5 -> 191.1 mm, vias 8 -> 164
- net /I2C5_SDA_M3: track 0.00 -> 170.9 mm
- net /I2C5_SCL_M3: track 0.00 -> 170.2 mm
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- added copper zone on B.Cu, net +12V
- added copper zone on F.Cu, net +12V
- added copper zone on B.Cu, net GND
- added copper zone on F.Cu, net GND
- added copper zone on F.Cu, net Net-(U4-VIN)
- added copper zone on F.Cu, net Net-(U5-VIN)
Other:
- board text added: "12V"
- board text added: "3V3"
- board text added: "5V0"
- board text added: "ACT"
- board text added: "BOOT"
- board text added: "DEBUG"
- board text added: "GND"
- board text added: "POWER"
- board text added: "RESET"
- board text added: "RX"
- board text added: "TEMP"
- board text added: "TX"
- board text added: "UART"
- board text added: "USER"
