File: OPI CM5 Blade Board/OPI CM5 Blade board.kicad_sch (KiCad schematic)
At the start: 16 parts, among them J1 OPi_CM5_CORE JP1 100PIN, J2 OPi_CM5_CORE JP2 100PIN, J3 OPi_CM5_CORE JP13100PIN, J4 Bus_PCI_Express_x4, J5 J_1-2199230-5, Q1 2SK3018, U1 SHT40-BD1B-R3, U2 SHT40-BD1B-R3

Commit message: LED SW added in schematic
Parts:
- added C2: 10μF, symbol OPI_CM5_Capacitor_SMD:C_Small
- added C27, C3 (x2), C4, C5, C6, CC1: 100nF, symbol OPI_CM5_Capacitor_SMD:C_Small
- added D1: D5819WS, Diode_SMD:D_SOD-323, symbol OPI_CM5_DIODE:B5819WS
- added D10, D11, D6, D7, D8, D9: BLU, symbol Device:LED_Small_Filled
- added D17, D2 (x2), D4: JEB05DFA, OPI_CM5_TVS_DIODE:DFN1006-2, symbol OPI_CM5_TVS_DIODE:ESD5341N
- added D3: RED, symbol Device:LED_Small_Filled
- added D5: GRN, symbol Device:LED_Small_Filled
- added ED5, ED6: ESD5341N, OPI_CM5_TVS_DIODE:DFN1006-2, symbol OPI_CM5_TVS_DIODE:ESD5341N
- added J2PIN_1R25: FAN, symbol Connector_Generic:Conn_01x02
- added NC/SIP1X3: SIP1X3, symbol Connector_Generic:Conn_01x03
- added Q2: 2SK3018, Package_TO_SOT_SMD:SOT-323_SC-70, symbol OPI_CM5_MOSFET:WNM6002-3/TR
- added R10, R13, R4, R6, R7, R8: 470R, symbol OPI_CM5_Resistor_SMD:R_Small
- added R11, R12: 0R, symbol OPI_CM5_Resistor_SMD:R_Small
- added R139, R14: 100R, symbol OPI_CM5_Resistor_SMD:R_Small
- added R144, R2: 200R, symbol OPI_CM5_Resistor_SMD:R_Small
- added R3: 560R, symbol OPI_CM5_Resistor_SMD:R_Small
- added R5: 1K, symbol OPI_CM5_Resistor_SMD:R_Small
- added R9: 10K, symbol OPI_CM5_Resistor_SMD:R_Small
- added SW1: USER_SW, symbol Switch:SW_Push
- added SW2: RESET_SW, symbol Switch:SW_Push
- added SW3: BOOT_SW, symbol Switch:SW_Push
- added SW4: PWR_SW, symbol Switch:SW_Push
Connections:
- net GND: now also C2.2, C27.2, C3.2, C3.2, C5.2, C6.2, CC1.2, D10.2 (A), D11.2 (A), D17.1 (A1), D2.1 (A1), D2.1 (A1), D3.2 (A), D4.1 (A1), D5.2 (A), D6.2 (A), D7.2 (A), D8.2 (A), D9.2 (A), ED5.1 (A1), ED6.1 (A1), NC/SIP1X3.1 (Pin_1), Q2.2 (S), SW1.1, SW2.1, SW3.1, SW4.1
- net GPIO3_C6: now also R144.1
- net GPIO4_B6: now also R9.1
- net PMIC_RESET_L: now also R14.1
- net PWRON_L: now also R2.1
- new net: C6.1, D17.2 (A2), R14.2, SW2.2
- new net: ED6.2 (A2), NC/SIP1X3.3 (Pin_3), R11.2
- new net: D8.1 (K), R7.2
- new net: D10.1 (K), R10.2
- new net: ED5.2 (A2), NC/SIP1X3.2 (Pin_2), R12.2
- new net: D6.1 (K), R5.2
- new net: D11.1 (K), R13.2
- new net: C3.1, D2.2 (A2), R139.2, SW3.2
- new net: D3.1 (K), R3.2
- new net: D9.1 (K), R8.2
- new net: C27.1, D4.2 (A2), R144.2, SW1.2
- new net: CC1.1, D2.2 (A2), R2.2, SW4.2
- new net: D7.1 (K), R6.2
- new net: D1.2 (A), J2PIN_1R25.2 (Pin_2), Q2.3 (D)
- new net: D5.1 (K), R4.2
- new net BOOT_KEY: R8.1
- new net BOOT_SW: R139.1
- new net DEBUG: R6.1
- new net POWER_KEY: R13.1
- new net PWM13_M1: C5.1, Q2.1 (G), R9.2
- new net RESET_KEY: R10.1
- new net UART_RX: R12.1
- new net UART_TX: R11.1
- new net USER_KEY: R7.1
- new net VCC_12V: R5.1
- new net VCC_3V3: R4.1
- new net VCC_5V0: C2.1, C3.1, D1.1 (K), J2PIN_1R25.1 (Pin_1), R3.1
Other:
- note added: "FAN CONTROL"
- note added: "MASKROM"
- note added: "PWR"
- note added: "RESET"
- note added: "UART DEBUG"
- note added: "USER_KEY"
- moved on the sheet: C1, C2, D1, H1, H2, H3, H4, Q1, R1

Commit message: Docs added
Other:
- note added: "01. HDMI0_TX0N 02. HDMI0_TX0P 03. HDMI0_TX1N 04. HDMI0_TX1P 05. HDMI0_TX2N 06. HDMI0_TX3P 07. HDMI0_TX2P 08. HDMI0_TX3N 09. HDMI_TX0_SCL_M0 10. HDMI_TX0_SDA_M0 11. HDMI_TX0_CEC_M0 12. HDMI0_TX_ON_H 13. HDMI0_SBDP 14. HDMI0_SBDP"
- note added: "10M/100M/1000M ETH"
- note added: "12V POWER"
- note added: "15. USB20_HOST0_DM 16. USB20_HOST0_DP"
- note added: "17. TYPEC0_USB20_OTG_DM 18. TYPEC0_USB20_OTG_DP"
- note added: "19. GMAC_MCLK/PWM13 20. GMAC_MDIO 21. GMAC_MDC 22. GMAC_RXCLK/SDIO_CLK 23. GMAC_RXDV/MIPI_CLK4/PWM2 24. GMAC_RXD0/MIPI_CLK2/PWM8 25. GMAC_RXD1/MIPI_CLK3/PWM9 26. GMAC_RXD2/SDIO_D2 27. GMAC_RXD3/SDIO_D3 28. GMAC_RXD3/SDIO_D3 29. GMAC_TXEN/PWM12 30. GMAC_TXD0 31. GMAC_TXD1 32. GMAC_TXD2/SDIO_D0 33. GMAC_TXD3/SDIO_D1 34. GPIO1-C0 35. GPIO1-C1"
- note added: "36. PCIE20_0_RXN 37. PCIE20_0_RXP 38. PCIE20_0_TXN 39. PCIE20_0_TXP 40. PCIE20_0_REFCLKN 41. PCIE20_0_REFCLKP 42. PCIE20x1_2_PERSTn_M0 43. PCIE20x1_2_CLKREQn_M0 44. PCIE20x1_2_WAKEn_M0 45. DAS/DSS (ACTIVITY LED)"
- note added: "46. UART_TX 47. UART_RX"
- note added: "48. PMIC_RESET_L"
- note added: "49. +12V 50. GND"
- note added: "HDMI2.1 TX0"
- note added: "M.2 NVME SSD"
- note added: "RESET BUTTON"
- note added: "UART"
- note added: "USB2.0"
- note added: "USB3.0 HOST"
Changed lines of the file:
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@@
 	(generator_version "9.0")
 	(paper "A3")
+	(text "17. TYPEC0_USB20_OTG_DM\n18. TYPEC0_USB20_OTG_DP"
+		(exclude_from_sim no)
+		(at 442.976 182.118 0)
+		(effects
+			(font
+				(size 1.27 1.27)
+			)
+			(justify left)
+		)
+	)
+	(text "48. PMIC_RESET_L"
+		(exclude_from_sim no)
+		(at 444.5 266.954 0)
+		(effects
+			(font
+				(size 1.27 1.27)
+			)
+			(justify left)
+		)
+	)
 	(text "PWR"
 		(exclude_from_sim no)
@@
 		)
 	)
+	(text "15. USB20_HOST0_DM\n16. USB20_HOST0_DP"
+		(exclude_from_sim no)
+		(at 442.722 173.228 0)
+		(effects
+			(font
+				(size 1.27 1.27)
+			)
+			(justify left)
+		)
+	)
+	(text "M.2 NVME SSD"
+		(exclude_from_sim no)
+		(at 443.484 228.092 0)
+		(effects
+			(font
+				(size 2.54 2.54)
+				(thickness 0.254)
+				(bold yes)
+			)
+			(justify left)
+		)
+	)
+	(text "19. GMAC_MCLK/PWM13\n20. GMAC_MDIO\n21. GMAC_MDC\n22. GMAC_RXCLK/SDIO_CLK\n23. GMAC_RXDV/MIPI_CLK4/PWM2\n24. GMAC_RXD0/MIPI_CLK2/PWM8\n25. GMAC_RXD1/MIPI_CLK3/PWM9\n26. GMAC_RXD2/SDIO_D2\n27. GMAC_RXD3/SDIO_D3\n28. GMAC_RXD3/SDIO_D3\n29. GMAC_TXEN/PWM12\n30. GMAC_TXD0\n31. GMAC_TXD1\n32. GMAC_TXD2/SDIO_D0\n33. GMAC_TXD3/SDIO_D1\n34. GPIO1-C0\n35. GPIO1-C1\n"
+		(exclude_from_sim no)
+		(at 443.738 206.248 0)
+		(effects
+			(font
+				(size 1.27 1.27)
+			)
+			(justify left)
+		)
+	)
 	(text "RESET"
 		(exclude_from_sim no)
@@
 		)
 	)
+	(text "HDMI2.1 TX0"
+		(exclude_from_sim no)
+		(at 454.152 128.016 0)
+		(effects
+			(font
+				(size 2.54 2.54)
+				(thickness 0.254)
+				(bold yes)
+			)
+		)
+	)
+	(text "10M/100M/1000M ETH"
+		(exclude_from_sim no)
+		(at 442.976 187.198 0)
+		(effects
+			(font
+				(size 2.54 2.54)
+				(thickness 0.254)
+				(bold yes)
+			)
+			(justify left)
+		)
+	)
+	(text "USB3.0 HOST\n"
+		(exclude_from_sim no)
+		(at 442.722 178.054 0)
+		(effects
+			(font
+				(size 2.54 2.54)
+				(thickness 0.254)
+				(bold yes)
+			)
+			(justify left)
+		)
+	)
+	(text "USB2.0\n"
+		(exclude_from_sim no)
+		(at 442.468 169.164 0)
+		(effects
+			(font
+				(size 2.54 2.54)
+				(thickness 0.254)
+				(bold yes)
+			)
+			(justify left)
+		)
+	)
+	(text "49. +12V\n50. GND"
+		(exclude_from_sim no)
+		(at 445.262 274.828 0)
+		(effects
+			(font
+				(size 1.27 1.27)
+			)
+			(justify left)
+		)
+	)
 	(text "OrangePI CM5\nCompute Module"
 		(exclude_from_sim no)
@@
 		)
 	)
+	(text "12V POWER"
+		(exclude_from_sim no)
+		(at 445.008 271.526 0)
+		(effects
+			(font
+				(size 2.54 2.54)
+				(thickness 0.254)
+				(bold yes)
+			)
+			(justify left)
+		)
+	)
+	(text "UART"
+		(exclude_from_sim no)
+		(at 444.246 254.508 0)
+		(effects
+			(font
+				(size 2.54 2.54)
+				(thickness 0.254)
+				(bold yes)
+			)
+			(justify left)
+		)
+	)
+	(text "36. PCIE20_0_RXN\n37. PCIE20_0_RXP\n38. PCIE20_0_TXN\n39. PCIE20_0_TXP\n40. PCIE20_0_REFCLKN\n41. PCIE20_0_REFCLKP\n42. PCIE20x1_2_PERSTn_M0\n43. PCIE20x1_2_CLKREQn_M0\n44. PCIE20x1_2_WAKEn_M0\n45. DAS/DSS (ACTIVITY LED)"
+		(exclude_from_sim no)
+		(at 444.246 239.776 0)
+		(effects
+			(font
+				(size 1.27 1.27)
+			)
+			(justify left)
+		)
+	)
 	(text "MASKROM\n"
 		(exclude_from_sim no)
@@
 		)
 	)
+	(text "RESET BUTTON"
+		(exclude_from_sim no)
+		(at 444.246 264.414 0)
+		(effects
+			(font
+				(size 2.54 2.54)
+				(thickness 0.254)
+				(bold yes)
+			)
+			(justify left)
+		)
+	)
 	(text "UART DEBUG\n"
 		(exclude_from_sim no)
@@
 		)
 	)
+	(text "01. HDMI0_TX0N\n02. HDMI0_TX0P\n03. HDMI0_TX1N\n04. HDMI0_TX1P\n05. HDMI0_TX2N\n06. HDMI0_TX3P\n07. HDMI0_TX2P\n08. HDMI0_TX3N\n\n09. HDMI_TX0_SCL_M0\n10. HDMI_TX0_SDA_M0\n11. HDMI_TX0_CEC_M0\n\n12. HDMI0_TX_ON_H\n\n13. HDMI0_SBDP\n14. HDMI0_SBDP"
+		(exclude_from_sim no)
+		(at 442.214 147.32 0)
+		(effects
+			(font
+				(size 1.27 1.27)
+			)
+			(justify left)
+		)
+	)
+	(text "46. UART_TX\n47. UART_RX"
+		(exclude_from_sim no)
+		(at 444.5 258.572 0)
+		(effects
+			(font
+				(size 1.27 1.27)
+			)
+			(justify left)
+		)
+	)

Commit message: Working on M.2 SSD
Parts:
- renumbered C2 to C22, C3 to C33, D1 to D22, D2 to D33
Connections:
- net USB20_HOST1_DM is gone; now on net USB20_HOST1_DN: J3.3 (Pin_3)
- net USB20_HOST1_DP: now also J4.B14 (PETp0)
- net USB20_HOST1_DN: now reaches J4.B15 (PETn0)
- net GPIO3_A0 renamed GMAC_TXD2
- net GPIO3_A1 renamed GMAC_TXD3
- net GPIO3_A2 renamed GMAC_RXD2
- net GPIO3_A3 renamed GMAC_RXD3
- net GPIO3_A4 renamed GMAC_TXCLK
- net GPIO3_A5 renamed GMAC_RXCLK
- net GPIO3_A7 renamed GMAC_RXD0
- net GPIO3_B0 renamed GMAC_RXD1
- net GPIO3_B1 renamed GMAC_RXDV
- net GPIO3_B3 renamed GMAC_TXD0
- net GPIO3_B4 renamed GMAC_TXD1
- net GPIO3_B5 renamed GMAC_TXEN
- net GPIO3_B6 renamed GMAC_MCLK/PWM13
- net GPIO3_C2 renamed GMAC_MDC
- net GPIO3_C3 renamed GMAC_MDIO
- net GPIO3_C7 renamed PCIE20x1_2_CLKREQn_M0
- net GPIO3_D0 renamed PCIE20x1_2_WAKEn_M0
- net GPIO3_D1 renamed PCIE20x1_2_PERSTn_M0
- net GPIO4_B5 renamed HDMI0_TX_ON_H
Changed lines of the file:
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@@
 	(wire
 		(pts
+			(xy 219.71 71.12) (xy 237.49 71.12)
+		)
+		(stroke
+			(width 0)
+			(type default)
+		)
+	)
+	(wire
+		(pts
 			(xy 16.51 83.82) (xy 30.48 83.82)
 		)
@@
 	(wire
 		(pts
-			(xy 151.13 73.66) (xy 171.45 73.66)
+			(xy 149.86 73.66) (xy 171.45 73.66)
 		)
 		(stroke
@@
 	(wire
 		(pts
+			(xy 219.71 73.66) (xy 237.49 73.66)
+		)
+		(stroke
+			(width 0)
+			(type default)
+		)
+	)
+	(wire
+		(pts
 			(xy 241.3 219.71) (xy 259.08 219.71)
 		)
@@
 	(wire
 		(pts
-			(xy 184.15 45.72) (xy 203.2 45.72)
+			(xy 184.15 45.72) (xy 208.28 45.72)
 		)
 		(stroke
@@
 	(wire
 		(pts
-			(xy 184.15 48.26) (xy 203.2 48.26)
+			(xy 184.15 48.26) (xy 208.28 48.26)
 		)
 		(stroke
@@
 		)
 	)
+	(label "USB20_HOST1_DP"
+		(at 219.71 71.12 0)
+		(effects
+			(font
+				(size 1.27 1.27)
+			)
+			(justify left bottom)
+		)
+		(property "Netclass" "USB"
+			(at 215.138 71.12 0)
+			(effects
+				(font
+					(size 1.27 1.27)
+					(italic yes)
+				)
+				(justify left)
+			)
+		)
+	)
 	(label "GND"
 		(at 68.58 88.9 0)
@@
 		)
 	)
-	(label "GPIO3_B5"
+	(label "GMAC_TXEN"
 		(at 151.13 83.82 0)
 		(effects
@@
 		)
 	)
+	(label "USB20_HOST1_DN"
+		(at 219.71 73.66 0)
+		(effects
+			(font
+				(size 1.27 1.27)
+			)
+			(justify left bottom)
+		)
+		(property "Netclass" "USB"
+			(at 215.138 73.66 0)
+			(effects
+				(font
+					(size 1.27 1.27)
+					(italic yes)
+				)
+				(justify left)
+			)
+		)
+	)
 	(label "GND"
 		(at 203.2 33.02 180)
@@
 		)
 	)
-	(label "GPIO3_A0"
+	(label "GMAC_TXD2"
 		(at 151.13 78.74 0)
 		(effects
@@
 		)
 	)
-	(label "GPIO3_D0"
-		(at 151.13 73.66 0)
+	(label "PCIE20x1_2_WAKEn_M0"
+		(at 149.86 73.66 0)
 		(effects
 			(font
@@
 		)
 	)
-	(label "GPIO3_D1"
-		(at 203.2 48.26 180)
+	(label "PCIE20x1_2_PERSTn_M0"
+		(at 208.28 48.26 180)
 		(effects
 			(font
@@
 		)
 	)
-	(label "GPIO3_A5"
+	(label "GMAC_RXCLK"
 		(at 203.2 91.44 180)
 		(effects
@@
 		)
 	)
-	(label "GPIO3_C3"
+	(label "GMAC_MDIO"
 		(at 151.13 86.36 0)
 		(effects
@@
 		)
 	)
-	(label "GPIO4_B5"
+	(label "HDMI0_TX_ON_H"
 		(at 68.58 81.28 0)
 		(effects
@@
 		)
 	)
-	(label "GPIO3_A1"
+	(label "GMAC_TXD3"
 		(at 203.2 71.12 180)
 		(effects
@@
 		)
 	)
-	(label "GPIO3_B1"
+	(label "GMAC_RXDV"
 		(at 151.13 93.98 0)
 		(effects
@@
 		)
 	)
-	(label "GPIO3_A3"
+	(label "GMAC_RXD3"
 		(at 151.13 99.06 0)
 		(effects
@@
 		)
 	)
-	(label "GPIO3_A4"
+	(label "GMAC_TXCLK"
 		(at 203.2 96.52 180)
 		(effects
@@
 		)
 	)
-	(label "GPIO3_C7"
-		(at 203.2 45.72 180)
+	(label "PCIE20x1_2_CLKREQn_M0"
+		(at 208.28 45.72 180)
 		(effects
 			(font
@@
 		)
 	)
-	(label "GPIO3_B6"
+	(label "GMAC_MCLK{slash}PWM13"
 		(at 151.13 91.44 0)
 		(effects
@@
 		)
 	)
-	(label "GPIO3_B3"
+	(label "GMAC_TXD0"
 		(at 203.2 76.2 180)
 		(effects
@@
 		)
 	)
-	(label "GPIO3_A7"
+	(label "GMAC_RXD0"
 		(at 203.2 93.98 180)
 		(effects
@@
 		)
 	)
-	(label "GPIO3_B4"
+	(label "GMAC_TXD1"
 		(at 151.13 81.28 0)
 		(effects
@@
 		)
 	)
-	(label "GPIO3_B0"
+	(label "GMAC_RXD1"
 		(at 203.2 88.9 180)
 		(effects
@@
 		)
 	)
-	(label "USB20_HOST1_DM"
+	(label "USB20_HOST1_DN"
 		(at 151.13 22.86 0)
 		(effects
@@
 		)
 	)
-	(label "GPIO3_C2"
+	(label "GMAC_MDC"
 		(at 151.13 134.62 0)
 		(effects
@@
 		)
 	)
-	(label "GPIO3_A2"
+	(label "GMAC_RXD2"
 		(at 151.13 96.52 0)
 		(effects
@@
 		(dnp no)
 		(fields_autoplaced yes)
-		(property "Reference" "C2"
+		(property "Reference" "C22"
 			(at 82.55 257.8162 0)
 			(effects
@@
 			(project "OPI CM5 Blade board"
 				(path "/18693405-0ee8-4c94-b62a-0ed8ec66960d"
-					(reference "C2")
+					(reference "C22")
 					(unit 1)
 				)
@@
 		(dnp no)
 		(fields_autoplaced yes)
-		(property "Reference" "C3"
+		(property "Reference" "C33"
 			(at 360.68 222.2562 0)
 			(effects
@@
 			(project "OPI CM5 Blade board"
 				(path "/18693405-0ee8-4c94-b62a-0ed8ec66960d"
-					(reference "C3")
+					(reference "C33")
 					(unit 1)
 				)
@@
 		(dnp no)
 		(fields_autoplaced yes)
-		(property "Reference" "D1"
+		(property "Reference" "D22"
 			(at 123.19 259.08 0)
 			(effects
@@
 			(project ""
 				(path "/18693405-0ee8-4c94-b62a-0ed8ec66960d"
-					(reference "D1")
+					(reference "D22")
 					(unit 1)
 				)
@@
 		(on_board yes)
 		(dnp no)
-		(property "Reference" "D2"
+		(property "Reference" "D33"
 			(at 268.224 244.094 90)
 			(effects
@@
 			(project "OPI CM5 Blade board"
 				(path "/18693405-0ee8-4c94-b62a-0ed8ec66960d"
-					(reference "D2")
+					(reference "D33")
 					(unit 1)
 				)

Commit message: M.2 SSD schematic complete
Parts:
- added C43: 47μF, symbol OPI_CM5_Capacitor_SMD:C_Small
- added C7, C8, C9: 100nF, symbol OPI_CM5_Capacitor_SMD:C_Small
- added D12: BLU, symbol Device:LED_Small_Filled
- added R15, R16, R17: 4.7K, symbol OPI_CM5_Resistor_SMD:R_Small
- added R18: 470R, symbol OPI_CM5_Resistor_SMD:R_Small
- added R19, R20, R21, R22: 4K7, symbol OPI_CM5_Resistor_SMD:R_Small
- added U3: TXB0304RUTR, OPI_CM5_Level_Shifter:RUT0012A, symbol OPI_CM5_Level_Shifter:TXB0304RUTR
- C40: renamed from C22; value C_Small -> 47μF; Rated Voltage 10V -> 6.3V
Connections:
- net GND: now also C40.2, J5.1 (CONFIG_3), J5.15 (GND), J5.21 (CONFIG_0), J5.27 (GND), J5.3 (GND), J5.33 (GND), J5.39 (GND), J5.45 (GND), J5.51 (GND), J5.57 (GND), J5.71 (GND), J5.73 (GND), J5.75 (CONFIG_2), J5.80 (GND), J5.9 (GND), J5.S1 (GND), J5.S2 (GND), C43.2, U3.6 (GND)
- net PCIE20_0_REFCLKN: now also J5.53 (REFCLKN)
- net PCIE20_0_REFCLKP: now also J5.55 (REFCLKP)
- net PCIE20_0_RXN: now also J5.41 (SATA_B+/PERN0)
- net PCIE20_0_RXP: now also J5.43 (SATA_B-/PERP0)
- net PCIE20_0_TXN: now also C8.2
- net PCIE20_0_TXP: now also C9.2
- net PCIE20x1_2_CLKREQn_M0: now also J5.52 (~{CLKREQ}), R21.1, U3.3 (A2), U3.9 (B2)
- net PCIE20x1_2_PERSTn_M0: now also J5.50 (~{PERST}), R22.1, U3.10 (B1), U3.2 (A1)
- net PCIE20x1_2_WAKEn_M0: now also J5.54 (~{PEWAKE}), R20.1, U3.4 (A3), U3.8 (B3)
- net VCC_1V8_S3: now also R19.2, U3.1 (VCCA)
- net VCC_3V3_S3: now also C40.1, J5.12 (VCC_3.3), J5.14 (VCC_3.3), J5.16 (VCC_3.3), J5.18 (VCC_3.3), J5.2 (VCC_3.3), J5.4 (VCC_3.3), J5.70 (VCC_3.3), J5.72 (VCC_3.3), J5.74 (VCC_3.3), C43.1, R18.1, R20.2, R21.2, R22.2, U3.11 (VCCB)
- net at J5.10 (DAS/DSS): now also D12.2 (A)
- net at J5.47 (SATA_A-/PETN0): now also C8.1
- net at J5.49 (SATA_A+/PETP0): now also C9.1
- new net: R19.1, U3.12 (OE)
- new net: D12.1 (K), R18.2
- no-connect marks 0 -> 36
Other:
- moved on the sheet: C40, J4

Commit message: New M.2 Symbol complete
Parts:
- removed C8, C9: 100nF, symbol OPI_CM5_Capacitor_SMD:C_Small
- removed D12: BLU, symbol Device:LED_Small_Filled
- removed R18: 470R, symbol OPI_CM5_Resistor_SMD:R_Small
- removed R20, R21, R22: 4K7, symbol OPI_CM5_Resistor_SMD:R_Small
- added C10, C11: 100nF, symbol OPI_CM5_Capacitor_SMD:C_Small
- added J6: Bus_PCI_Express_x4, Connector_PCBEdge:BUS_PCIexpress_x4, symbol OPI_CM5_PCIe_CONN:Bus_PCI_Express_x4
- added R23, R24, R25: 4K7, symbol OPI_CM5_Resistor_SMD:R_Small
- C27, C3, C6, CC1: footprint (none) -> Capacitor_SMD:C_0201_0603Metric_Pad0.64x0.40mm_HandSolder
- D10, D11, D3, D5, D6, D7, D8, D9: footprint (none) -> LED_SMD:LED_0603_1608Metric_Pad1.05x0.95mm_HandSolder
- R10, R11, R12, R13, R139, R14, R144, R2, R3, R4, R5, R6, R7, R8: footprint (none) -> Resistor_SMD:R_0201_0603Metric_Pad0.64x0.40mm_HandSolder
- SW1, SW2, SW3, SW4: footprint (none) -> OPI_CM5_PUSH_SW:SW4_PTS815 SJM 250 SMTR LFS_CNK; symbol Switch:SW_Push -> OPI_CM5_PUSH_SW:SW_Push
Connections:
- net GND: now also J5.69 (CONFIG_1), SW1.2, SW2.2, SW3.2, SW4.2
- net PCIE20_0_TXN: now also C11.2
- net PCIE20_0_TXP: now also C10.2
- net PCIE20x1_2_CLKREQn_M0: now also R24.1
- net PCIE20x1_2_PERSTn_M0: now also R23.1
- net PCIE20x1_2_WAKEn_M0: now also R25.1
- net VCC_3V3_S3: now also R23.2, R24.2, R25.2
- net at C6.1, D17.2 (A2), R14.2: now also SW2.3, SW2.4; no longer SW2.2
- net at C3.1, D33.2 (A2), R139.2: now also SW3.3, SW3.4; no longer SW3.2
- net at J5.49 (SATA_A+/PETP0): now also C10.1
- net at C27.1, D4.2 (A2), R144.2: now also SW1.3, SW1.4; no longer SW1.2
- net at J5.20 (N/A): now also J5.22 (N/A), J5.24 (N/A), J5.26 (N/A), J5.28 (N/A), J5.30 (N/A), J5.32 (N/A), J5.34 (N/A), J5.36 (N/A), J5.40 (N/A), J5.42 (N/A), J5.44 (N/A), J5.46 (N/A), J5.48 (N/A), J5.6 (N/A), J5.67 (N/A), J5.8 (N/A)
- net at J5.47 (SATA_A-/PETN0): now also C11.1
- net at CC1.1, D2.2 (A2), R2.2: now also SW4.3, SW4.4; no longer SW4.2
- no-connect marks 36 -> 20
Other:
- moved on the sheet: C4, C40, C43, C7, H1, H2, H3, H4, R19, U3
