File: OPI CM5 Blade Board/OPI CM5 Blade board.kicad_sch (KiCad schematic)
At the start: 74 parts, among them J1 OPi_CM5_CORE JP1 100PIN, J2 OPi_CM5_CORE JP2 100PIN, J2PIN_1R25 FAN, J3 OPi_CM5_CORE JP13100PIN, J4 Bus_PCI_Express_x4, J5 J_1-2199230-5, J6 Bus_PCI_Express_x4, Q1 2SK3018, Q2 2SK3018, SW1 USER_SW, SW2 RESET_SW, SW3 BOOT_SW, SW4 PWR_SW, U1 SHT40-BD1B-R3, U2 SHT40-BD1B-R3, U3 TXB0304RUTR

Commit message: Working on routing
Parts:
- removed C1: C_Small, symbol OPI_CM5_Capacitor_SMD:C_Small
- removed C2: 10μF, symbol OPI_CM5_Capacitor_SMD:C_Small
- removed C33, C4, C5: 100nF, symbol OPI_CM5_Capacitor_SMD:C_Small
- removed D1: D5819WS, Diode_SMD:D_SOD-323, symbol OPI_CM5_DIODE:B5819WS
- removed D22: D_TVS_Small_Filled, symbol Device:D_TVS_Small_Filled
- removed D5: GRN, LED_SMD:LED_0603_1608Metric_Pad1.05x0.95mm_HandSolder, symbol Device:LED_Small_Filled
- removed D6: BLU, LED_SMD:LED_0603_1608Metric_Pad1.05x0.95mm_HandSolder, symbol Device:LED_Small_Filled
- removed J2PIN_1R25: FAN, symbol Connector_Generic:Conn_01x02
- removed J4: Bus_PCI_Express_x4, Connector_PCBEdge:BUS_PCIexpress_x4, symbol Connector:Bus_PCI_Express_x4
- removed Q1: 2SK3018, Package_TO_SOT_SMD:SOT-323_SC-70, symbol OPI_CM5_MOSFET:2SK3018
- removed Q2: 2SK3018, Package_TO_SOT_SMD:SOT-323_SC-70, symbol OPI_CM5_MOSFET:WNM6002-3/TR
- removed R1: R_Small, symbol OPI_CM5_Resistor_SMD:R_Small
- removed R15, R16, R17: 4.7K, symbol OPI_CM5_Resistor_SMD:R_Small
- removed R9: 10K, symbol OPI_CM5_Resistor_SMD:R_Small
- added C12, C14, C15, C20: 10μF, Capacitor_SMD:C_0805_2012Metric_Pad1.18x1.45mm_HandSolder, symbol OPI_CM5_Capacitor_SMD:C_Small
- added C13, C19: 22μF, Capacitor_SMD:C_0805_2012Metric_Pad1.18x1.45mm_HandSolder, symbol OPI_CM5_Capacitor_SMD:C_Small
- added C16, CC2, CC3, CC4, CC5, CC6, CC7: 100nF, Capacitor_SMD:C_0201_0603Metric_Pad0.64x0.40mm_HandSolder, symbol OPI_CM5_Capacitor_SMD:C_Small
- added C17, C8: 22pF, Capacitor_SMD:C_0201_0603Metric_Pad0.64x0.40mm_HandSolder, symbol OPI_CM5_Capacitor_SMD:C_Small
- added C18, C9: 47μF, Capacitor_SMD:C_0805_2012Metric_Pad1.18x1.45mm_HandSolder, symbol OPI_CM5_Capacitor_SMD:C_Small
- added L1, L2: WPN4020H2R2MT, OPI_CM5_INDUCTOR_SMD:WPN4020H2R2MT, symbol OPI_CM5_INDUCTOR_SMD:WPN4020H2R2MT
- added R18, R20, R21, R22: 100K, Resistor_SMD:R_0201_0603Metric_Pad0.64x0.40mm_HandSolder, symbol OPI_CM5_Resistor_SMD:R_Small
- added R26: 110K, Resistor_SMD:R_0201_0603Metric_Pad0.64x0.40mm_HandSolder, symbol OPI_CM5_Resistor_SMD:R_Small
- added R27: 15K, Resistor_SMD:R_0201_0603Metric_Pad0.64x0.40mm_HandSolder, symbol OPI_CM5_Resistor_SMD:R_Small
- added U4, U5: SM8103ADC, Package_TO_SOT_SMD:SOT-23-6_Handsoldering, symbol OPI_CM5_REGULATOR_SWITCHING:SM8103ADC
- C10, C11, C7: footprint (none) -> Capacitor_SMD:C_0201_0603Metric_Pad0.64x0.40mm_HandSolder
- C40, C43: footprint (none) -> Capacitor_SMD:C_0805_2012Metric_Pad1.18x1.45mm_HandSolder
- D10, D9: value BLU -> YLO
- D7: value BLU -> ORN
- D8: value BLU -> GRN
- NC/SIP1X3: footprint (none) -> Connector_PinHeader_1.00mm:PinHeader_1x03_P1.00mm_Vertical_SMD_Pin1Right
- R19: footprint (none) -> Resistor_SMD:R_0201_0603Metric_Pad0.64x0.40mm_HandSolder; now not fitted; now left out of the parts list
- R23, R24, R25: footprint (none) -> Resistor_SMD:R_0201_0603Metric_Pad0.64x0.40mm_HandSolder
- R4: value 470R -> 100K; Tolarance 5% -> 1%
- R5: value 1K -> 22.1K; Tolarance 5% -> 1%
- U3: now not fitted; now left out of the parts list
- renumbered J6 to J4
Connections:
- net BOOT_SW is gone; now on net BOOT_KEY: R139.1
- net GMAC_MCLK/PWM13 is gone; now on net GMAC_MCLK: J3.57 (Pin_57)
- net GPIO0_C7 is gone; now on net DEBUG_LED: J3.79 (Pin_79)
- net GPIO0_D4 is gone; now on net POWER_KEY: J3.81 (Pin_81)
- net GPIO1_B6 is gone; now on net I2C5_SCL_M3: J1.41 (Pin_41)
- net GPIO1_B7 is gone; now on net I2C5_SDA_M3: J1.45 (Pin_45)
- net GPIO1_C0 is gone; now on net I2C3_SDA_M0: J1.24 (Pin_24)
- net GPIO1_C1 is gone; now on net I2C3_SCL_M0: J1.26 (Pin_26)
- net GPIO4_B6 is gone; now on net USER_KEY: J1.95 (Pin_95)
- net GPIO_VREF is gone; now on net VCC_3V3_S3: J1.78 (Pin_78)
- net RESET_KEY is gone; now on net TMP_SN2_LED: R10.1
- net SARADC_IN0 is gone; now on net BOOT_KEY: J1.93 (Pin_93)
- net VCC_12V is gone; now on net GND: R5.1
- net VCC_3V3 is gone; now on an unnamed net: R4.1
- net BOOT_KEY: no longer R8.1
- net GMAC_MDC: now also J4.A16
- net GMAC_MDIO: now also J4.A26
- net GMAC_RXCLK: now also J4.A19
- net GMAC_RXD0: now also J4.A18
- net GMAC_RXD1: now also J4.A20
- net GMAC_RXD2: now also J4.A29
- net GMAC_RXD3: now also J4.A30
- net GMAC_RXDV: now also J4.A28
- net GMAC_TXCLK: now also J4.A17
- net GMAC_TXD0: now also J4.A21
- net GMAC_TXD1: now also J4.A24
- net GMAC_TXD2: now also J4.A23
- net GMAC_TXD3: now also J4.A22
- net GMAC_TXEN: now also J4.A25
- net GND: now also J4.A14, J4.A4, J4.A7, J4.A9, J4.B14, J4.B17, J4.B4, J4.B7, J4.B9, U1.4 (VSS), U2.4 (VSS), C12.2, C13.2, C14.2, C15.2, C18.2, C19.2, C20.2, C9.2, CC2.2, CC3.2, CC4.2, CC5.2, CC6.2, CC7.2, R20.2, R22.2, R27.1, U4.2 (GND), U5.2 (GND)
- net GPIO3_C6: no longer R144.1
- net HDMI0_SBDP: now also J4.B32
- net HDMI0_TX_ON_H: now also J4.B18
- net HDMI_TX0_CEC_M0: now also J4.B19
- net HDMI_TX0_D0N: now also J4.B29
- net HDMI_TX0_D0P: now also J4.B30
- net HDMI_TX0_D1P: now also J4.B24
- net HDMI_TX0_D2N: now also J4.B23
- net HDMI_TX0_D2P: now also J4.B22
- net HDMI_TX0_D3N: now also J4.B27
- net HDMI_TX0_D3P: now also J4.B28
- net HDMI_TX0_SBDN: now also J4.B20
- net HDMI_TX0_SCL_M0: now also J4.B26
- net HDMI_TX0_SDA_M0: now also J4.B21
- net PCIE20x1_2_CLKREQn_M0: now also U3.4 (A3); no longer U3.3 (A2), U3.9 (B2)
- net PCIE20x1_2_PERSTn_M0: now also U3.3 (A2); no longer U3.10 (B1), U3.2 (A1)
- net PCIE20x1_2_WAKEn_M0: now also U3.2 (A1); no longer U3.4 (A3), U3.8 (B3)
- net PMIC_RESET_L: now also J4.A11
- net POWER_KEY: no longer R13.1
- net PWRON_L: now also J4.B11
- net UART_RX: now also J4.B13
- net UART_TX: now also J4.B12
- net USB20_HOST1_DP: now also J4.B16
- net USER_KEY: now also R144.1; no longer R7.1
- net VCC_3V3_S3: no longer C40.1, C43.1, J5.12 (VCC_3.3), J5.14 (VCC_3.3), J5.16 (VCC_3.3), J5.18 (VCC_3.3), J5.2 (VCC_3.3), J5.4 (VCC_3.3), J5.70 (VCC_3.3), J5.72 (VCC_3.3), J5.74 (VCC_3.3), R23.2, R24.2, R25.2
- net +12V: now reaches J4.A1
- net +12V: now also J4.A2, J4.A3, J4.B1, J4.B2, J4.B3, C14.1, C15.1, CC4.1, CC5.1, R18.1, R21.1, U4.1 (BS), U5.1 (BS)
- net +1.8V: now reaches J4.A10
- net +1.8V: now also J4.B10
- net GMAC_MCLK: now reaches J4.A27
- net +5V: now reaches J4.A5
- net +5V: now also J4.A6, J4.B5, J4.B6
- net +3.3V: now reaches J4.A8
- net +3.3V: now also J4.B8
- net USB20_HOST1_DM: now reaches J4.B15
- net HDMI0_TX1N: now reaches J4.B25
- net at R5.2: now also C8.2, U4.3 (FB)
- net at C7.1: now also U4.6 (LX)
- net at C7.2: now also L1.1, U4.5 (VIN)
- net I2C5_SDA_M3: now reaches U1.1 (SDA)
- net I2C5_SCL_M3: now reaches U1.2 (SCL)
- net +3.3V_3A: now reaches U1.3 (VDD)
- net +3.3V_3A: now also C40.1, C43.1, J5.12 (VCC_3.3), J5.14 (VCC_3.3), J5.16 (VCC_3.3), J5.18 (VCC_3.3), J5.2 (VCC_3.3), J5.4 (VCC_3.3), J5.70 (VCC_3.3), J5.72 (VCC_3.3), J5.74 (VCC_3.3), R23.2, R24.2, R25.2, R4.2, U2.3 (VDD), C12.1, C13.1, C8.1, C9.1, CC2.1, L1.2
- net I2C3_SDA_M0: now reaches U2.1 (SDA)
- net I2C3_SCL_M0: now reaches U2.2 (SCL)
- net M.2_ACT: now reaches J5.10 (DAS/DSS)
- net M.2_ACT: now also R13.1
- net DEBUG renamed DEBUG_LED
- net GPIO0_C4 renamed TMP_SN1_LED
- net TMP_SN1_LED: now also R8.1
- net GPIO0_D3 renamed TMP_SN2_LED
- net GPIO0_D5 renamed USER_LED
- net USER_LED: now also R7.1
- net VBUS renamed +5V_3A
- net +5V_3A: now also C17.1, C18.1, C19.1, C20.1, CC7.1, L2.2, R26.2
- new net: C17.2, R26.1, R27.2, U5.3 (FB)
- new net: CC3.1, R18.2, R20.1, U4.4 (EN)
- new net: CC6.1, R21.2, R22.1, U5.4 (EN)
- new net: C16.2, L2.1, U5.5 (VIN)
- new net: C16.1, U5.6 (LX)
- new net PCIE20x1_2_CLKREQn: U3.8 (B3)
- new net PCIE20x1_2_PERSTn: U3.9 (B2)
- new net PCIE20x1_2_WAKEn: U3.10 (B1)
- no-connect marks 20 -> 25
Other:
- note added: "*GPIO_VREF(PIN 78) IS CONECTED WITH VCC_3V3S3"
- note added: "*VBUS IS +5V_3A"
- note added: "+3.3V 3A"
- note added: "+5.0V 3A"
- note added: "DISPLAY LEDS"
- note added: "PCIe EDGE CONNECTOR"
- note added: "SWITCHES"
- note added: "TEMPARATURE SENSOR 1"
- note added: "TEMPARATURE SENSOR 2"
- note removed: "01. HDMI0_TX0N 02. HDMI0_TX0P 03. HDMI0_TX1N 04. HDMI0_TX1P 05. HDMI0_TX2N 06. HDMI0_TX3P 07. HDMI0_TX2P 08. HDMI0_TX3N 09. HDMI_TX0_SCL_M0 10. HDMI_TX0_SDA_M0 11. HDMI_TX0_CEC_M0 12. HDMI0_TX_ON_H 13. HDMI0_SBDP 14. HDMI0_SBDP"
- note removed: "10M/100M/1000M ETH"
- note removed: "12V POWER"
- note removed: "15. USB20_HOST0_DM 16. USB20_HOST0_DP"
- note removed: "17. TYPEC0_USB20_OTG_DM 18. TYPEC0_USB20_OTG_DP"
- note removed: "19. GMAC_MCLK/PWM13 20. GMAC_MDIO 21. GMAC_MDC 22. GMAC_RXCLK/SDIO_CLK 23. GMAC_RXDV/MIPI_CLK4/PWM2 24. GMAC_RXD0/MIPI_CLK2/PWM8 25. GMAC_RXD1/MIPI_CLK3/PWM9 26. GMAC_RXD2/SDIO_D2 27. GMAC_RXD3/SDIO_D3 28. GMAC_RXD3/SDIO_D3 29. GMAC_TXEN/PWM12 30. GMAC_TXD0 31. GMAC_TXD1 32. GMAC_TXD2/SDIO_D0 33. GMAC_TXD3/SDIO_D1 34. GPIO1-C0 35. GPIO1-C1"
- note removed: "36. PCIE20_0_RXN 37. PCIE20_0_RXP 38. PCIE20_0_TXN 39. PCIE20_0_TXP 40. PCIE20_0_REFCLKN 41. PCIE20_0_REFCLKP 42. PCIE20x1_2_PERSTn_M0 43. PCIE20x1_2_CLKREQn_M0 44. PCIE20x1_2_WAKEn_M0 45. DAS/DSS (ACTIVITY LED)"
- note removed: "46. UART_TX 47. UART_RX"
- note removed: "48. PMIC_RESET_L"
- note removed: "49. +12V 50. GND"
- note removed: "FAN CONTROL"
- note removed: "HDMI2.1 TX0"
- note removed: "RESET BUTTON"
- note removed: "UART"
- note removed: "USB2.0"
- note removed: "USB3.0 HOST"
- moved on the sheet: C10, C11, C27, C3, C40, C43, C6, C7, CC1, D10, D11, D17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

Commit message: Project complete
Parts:
- added C1, C2, C21, C22, C23, C24, C4, C5: 220nF, Capacitor_SMD:C_0201_0603Metric_Pad0.64x0.40mm_HandSolder, symbol OPI_CM5_Capacitor_SMD:C_Small
- added D1: RED, LED_SMD:LED_0603_1608Metric_Pad1.05x0.95mm_HandSolder, symbol Device:LED_Small_Filled
- added R1: 560R, Resistor_SMD:R_0201_0603Metric_Pad0.64x0.40mm_HandSolder, symbol OPI_CM5_Resistor_SMD:R_Small
Connections:
- net HDMI_TX0_D1N is gone; now on net HDMI0_TX1N: J2.78 (Pin_78)
- net UART_RX is gone; now on net UART2_RX: J4.B13, R12.1
- net UART_TX is gone; now on net UART2_TX: J4.B12, R11.1
- net USB20_HOST1_DM is gone; now on net USB20_HOST1_DN: J4.B15
- net VCC_5V0 is gone; now on net +5V_3A: R3.1
- net +12V: now also R10.1
- net +3.3V_3A: now also R1.1; no longer U2.3 (VDD)
- net GMAC_MDC: now also J4.A15; no longer J4.A16
- net GMAC_TXCLK: now also J4.A16; no longer J4.A17
- net GND: now also J4.A17, D1.2 (A)
- net HDMI0_SBDP: now also J4.B20; no longer J4.B32
- net HDMI0_TX1N: now also J4.B24, C22.1; no longer J4.B25
- net HDMI0_TX_ON_H: now also J4.B32; no longer J4.B18
- net TMP_SN2_LED: no longer R10.1
- net USB20_HOST1_DN: now also J3.1 (Pin_1); no longer J3.3 (Pin_3)
- net USB20_HOST1_DP: now also J3.3 (Pin_3); no longer J3.1 (Pin_1)
- net VCC_3V3_S3: now also U2.3 (VDD)
- net HDMI_TX0_CEC_M0 renamed HDMI0_SBDN
- net HDMI0_SBDN: now also J2.53 (Pin_53); no longer J2.51 (Pin_51)
- net HDMI_TX0_D0N renamed HDMI0_TX0N
- net HDMI0_TX0N: now also J4.B27, C5.1; no longer J4.B29
- net HDMI_TX0_D0P renamed HDMI0_TX0P
- net HDMI0_TX0P: now also J4.B28, C4.1; no longer J4.B30
- net HDMI_TX0_D1P renamed HDMI0_TX1P
- net HDMI0_TX1P: now also J4.B23, C21.1; no longer J4.B24
- net HDMI_TX0_D2N renamed HDMI0_TX2N
- net HDMI0_TX2N: now also J4.B29, C2.1; no longer J4.B23
- net HDMI_TX0_D2P renamed HDMI0_TX2P
- net HDMI0_TX2P: now also J4.B30, C1.1; no longer J4.B22
- net HDMI_TX0_D3N renamed HDMI0_TX3N
- net HDMI0_TX3N: now also J4.B26, C24.1; no longer J4.B27
- net HDMI_TX0_D3P renamed HDMI0_TX3P
- net HDMI0_TX3P: now also J4.B25, C23.1; no longer J4.B28
- removed net HDMI_TX0_SBDN: J2.53 (Pin_53), J4.B20
- net HDMI_TX0_SCL_M0 renamed HDMI0_TX_SCL_M0
- net HDMI0_TX_SCL_M0: now also J4.B22; no longer J4.B26
- net HDMI_TX0_SDA_M0 renamed HDMI0_TX_SDA_M0
- new net: D1.1 (K), R1.2
- new net HDMI0_PORT_TX0N: C5.2
- new net HDMI0_PORT_TX0P: C4.2
- new net HDMI0_PORT_TX1N: C22.2
- new net HDMI0_PORT_TX1P: C21.2
- new net HDMI0_PORT_TX2N: C2.2
- new net HDMI0_PORT_TX2P: C1.2
- new net HDMI0_PORT_TX3N: C24.2
- new net HDMI0_PORT_TX3P: C23.2
- new net HDMI0_TX_CEC_M0: J2.51 (Pin_51), J4.B18
- no-connect marks 25 -> 24
Other:
- moved on the sheet: D10, D11, D7, D8, D9, J4, R10, R13, R6, R7, R8
